File: EEMR TKL Keyboard/EEMR TKL Keyboard.sch (KiCad schematic (older format))
At the start: 192 parts, among them SW1 SW_Push, U1 ATmega32U4-AU, Y1 16MHz

Commit message: new projects
Parts:
- C1: renamed from C2; footprint (none) -> Capacitor_SMD:C_0805_2012Metric_Pad1.15x1.40mm_HandSolder
- C2: renamed from C1; footprint (none) -> Capacitor_SMD:C_0805_2012Metric_Pad1.15x1.40mm_HandSolder
- C3, C4, C5, C6, C7: footprint (none) -> Capacitor_SMD:C_0805_2012Metric_Pad1.15x1.40mm_HandSolder
- F1: footprint (none) -> Fuse:Fuse_1206_3216Metric_Pad1.42x1.75mm_HandSolder
- MX1, MX20, MX76: footprint (none) -> MX_Only:MXOnly-1U-NoLED; symbol MX_Alps_Hybrid:MX-NoLED -> EEMR-TKL-Keyboard-rescue:MX-NoLED-MX_Alps_Hybrid
- MX10: renamed from MX55; footprint (none) -> MX_Only:MXOnly-1U-NoLED; symbol MX_Alps_Hybrid:MX-NoLED -> EEMR-TKL-Keyboard-rescue:MX-NoLED-MX_Alps_Hybrid
- MX11: renamed from MX61; footprint (none) -> MX_Only:MXOnly-1U-NoLED; symbol MX_Alps_Hybrid:MX-NoLED -> EEMR-TKL-Keyboard-rescue:MX-NoLED-MX_Alps_Hybrid
- MX12: renamed from MX67; footprint (none) -> MX_Only:MXOnly-1U-NoLED; symbol MX_Alps_Hybrid:MX-NoLED -> EEMR-TKL-Keyboard-rescue:MX-NoLED-MX_Alps_Hybrid
- MX13: renamed from MX72; footprint (none) -> MX_Only:MXOnly-1U-NoLED; symbol MX_Alps_Hybrid:MX-NoLED -> EEMR-TKL-Keyboard-rescue:MX-NoLED-MX_Alps_Hybrid
- MX14: renamed from MX77; footprint (none) -> MX_Only:MXOnly-1U-NoLED; symbol MX_Alps_Hybrid:MX-NoLED -> EEMR-TKL-Keyboard-rescue:MX-NoLED-MX_Alps_Hybrid
- MX15: renamed from MX80; footprint (none) -> MX_Only:MXOnly-1U-NoLED; symbol MX_Alps_Hybrid:MX-NoLED -> EEMR-TKL-Keyboard-rescue:MX-NoLED-MX_Alps_Hybrid
- MX16: renamed from MX83; footprint (none) -> MX_Only:MXOnly-1U-NoLED; symbol MX_Alps_Hybrid:MX-NoLED -> EEMR-TKL-Keyboard-rescue:MX-NoLED-MX_Alps_Hybrid
- MX17: renamed from MX2; footprint (none) -> MX_Only:MXOnly-1U-NoLED; symbol MX_Alps_Hybrid:MX-NoLED -> EEMR-TKL-Keyboard-rescue:MX-NoLED-MX_Alps_Hybrid
- MX18: renamed from MX8; footprint (none) -> MX_Only:MXOnly-1U-NoLED; symbol MX_Alps_Hybrid:MX-NoLED -> EEMR-TKL-Keyboard-rescue:MX-NoLED-MX_Alps_Hybrid
- MX19: renamed from MX14; footprint (none) -> MX_Only:MXOnly-1U-NoLED; symbol MX_Alps_Hybrid:MX-NoLED -> EEMR-TKL-Keyboard-rescue:MX-NoLED-MX_Alps_Hybrid
- MX2: renamed from MX7; footprint (none) -> MX_Only:MXOnly-1U-NoLED; symbol MX_Alps_Hybrid:MX-NoLED -> EEMR-TKL-Keyboard-rescue:MX-NoLED-MX_Alps_Hybrid
- MX21: renamed from MX26; footprint (none) -> MX_Only:MXOnly-1U-NoLED; symbol MX_Alps_Hybrid:MX-NoLED -> EEMR-TKL-Keyboard-rescue:MX-NoLED-MX_Alps_Hybrid
- MX22: renamed from MX32; footprint (none) -> MX_Only:MXOnly-1U-NoLED; symbol MX_Alps_Hybrid:MX-NoLED -> EEMR-TKL-Keyboard-rescue:MX-NoLED-MX_Alps_Hybrid
- MX23: renamed from MX38; footprint (none) -> MX_Only:MXOnly-1U-NoLED; symbol MX_Alps_Hybrid:MX-NoLED -> EEMR-TKL-Keyboard-rescue:MX-NoLED-MX_Alps_Hybrid
- MX24: renamed from MX44; footprint (none) -> MX_Only:MXOnly-1U-NoLED; symbol MX_Alps_Hybrid:MX-NoLED -> EEMR-TKL-Keyboard-rescue:MX-NoLED-MX_Alps_Hybrid
- MX25: renamed from MX50; footprint (none) -> MX_Only:MXOnly-1U-NoLED; symbol MX_Alps_Hybrid:MX-NoLED -> EEMR-TKL-Keyboard-rescue:MX-NoLED-MX_Alps_Hybrid
- MX26: renamed from MX56; footprint (none) -> MX_Only:MXOnly-1U-NoLED; symbol MX_Alps_Hybrid:MX-NoLED -> EEMR-TKL-Keyboard-rescue:MX-NoLED-MX_Alps_Hybrid
- MX27: renamed from MX62; footprint (none) -> MX_Only:MXOnly-1U-NoLED; symbol MX_Alps_Hybrid:MX-NoLED -> EEMR-TKL-Keyboard-rescue:MX-NoLED-MX_Alps_Hybrid
- MX28: renamed from MX68; footprint (none) -> MX_Only:MXOnly-1U-NoLED; symbol MX_Alps_Hybrid:MX-NoLED -> EEMR-TKL-Keyboard-rescue:MX-NoLED-MX_Alps_Hybrid
- MX29: renamed from MX73; footprint (none) -> MX_Only:MXOnly-1U-NoLED; symbol MX_Alps_Hybrid:MX-NoLED -> EEMR-TKL-Keyboard-rescue:MX-NoLED-MX_Alps_Hybrid
- MX3: renamed from MX13; footprint (none) -> MX_Only:MXOnly-1U-NoLED; symbol MX_Alps_Hybrid:MX-NoLED -> EEMR-TKL-Keyboard-rescue:MX-NoLED-MX_Alps_Hybrid
- MX30: renamed from MX78; footprint (none) -> MX_Only:MXOnly-2U-NoLED; symbol MX_Alps_Hybrid:MX-NoLED -> EEMR-TKL-Keyboard-rescue:MX-NoLED-MX_Alps_Hybrid
- MX31: renamed from MX81; footprint (none) -> MX_Only:MXOnly-1U-NoLED; symbol MX_Alps_Hybrid:MX-NoLED -> EEMR-TKL-Keyboard-rescue:MX-NoLED-MX_Alps_Hybrid
- MX32: renamed from MX84; footprint (none) -> MX_Only:MXOnly-1U-NoLED; symbol MX_Alps_Hybrid:MX-NoLED -> EEMR-TKL-Keyboard-rescue:MX-NoLED-MX_Alps_Hybrid
- MX33: renamed from MX86; footprint (none) -> MX_Only:MXOnly-1U-NoLED; symbol MX_Alps_Hybrid:MX-NoLED -> EEMR-TKL-Keyboard-rescue:MX-NoLED-MX_Alps_Hybrid
- MX34: renamed from MX3; footprint (none) -> MX_Only:MXOnly-1.5U-NoLED; symbol MX_Alps_Hybrid:MX-NoLED -> EEMR-TKL-Keyboard-rescue:MX-NoLED-MX_Alps_Hybrid
- MX35: renamed from MX9; footprint (none) -> MX_Only:MXOnly-1U-NoLED; symbol MX_Alps_Hybrid:MX-NoLED -> EEMR-TKL-Keyboard-rescue:MX-NoLED-MX_Alps_Hybrid
- MX36: renamed from MX15; footprint (none) -> MX_Only:MXOnly-1U-NoLED; symbol MX_Alps_Hybrid:MX-NoLED -> EEMR-TKL-Keyboard-rescue:MX-NoLED-MX_Alps_Hybrid
- MX37: renamed from MX21; footprint (none) -> MX_Only:MXOnly-1U-NoLED; symbol MX_Alps_Hybrid:MX-NoLED -> EEMR-TKL-Keyboard-rescue:MX-NoLED-MX_Alps_Hybrid
- MX38: renamed from MX27; footprint (none) -> MX_Only:MXOnly-1U-NoLED; symbol MX_Alps_Hybrid:MX-NoLED -> EEMR-TKL-Keyboard-rescue:MX-NoLED-MX_Alps_Hybrid
- MX39: renamed from MX33; footprint (none) -> MX_Only:MXOnly-1U-NoLED; symbol MX_Alps_Hybrid:MX-NoLED -> EEMR-TKL-Keyboard-rescue:MX-NoLED-MX_Alps_Hybrid
- MX4: renamed from MX19; footprint (none) -> MX_Only:MXOnly-1U-NoLED; symbol MX_Alps_Hybrid:MX-NoLED -> EEMR-TKL-Keyboard-rescue:MX-NoLED-MX_Alps_Hybrid
- MX40: renamed from MX39; footprint (none) -> MX_Only:MXOnly-1U-NoLED; symbol MX_Alps_Hybrid:MX-NoLED -> EEMR-TKL-Keyboard-rescue:MX-NoLED-MX_Alps_Hybrid
- MX41: renamed from MX45; footprint (none) -> MX_Only:MXOnly-1U-NoLED; symbol MX_Alps_Hybrid:MX-NoLED -> EEMR-TKL-Keyboard-rescue:MX-NoLED-MX_Alps_Hybrid
- MX42: renamed from MX51; footprint (none) -> MX_Only:MXOnly-1U-NoLED; symbol MX_Alps_Hybrid:MX-NoLED -> EEMR-TKL-Keyboard-rescue:MX-NoLED-MX_Alps_Hybrid
- MX43: renamed from MX57; footprint (none) -> MX_Only:MXOnly-1U-NoLED; symbol MX_Alps_Hybrid:MX-NoLED -> EEMR-TKL-Keyboard-rescue:MX-NoLED-MX_Alps_Hybrid
- MX44: renamed from MX63; footprint (none) -> MX_Only:MXOnly-1U-NoLED; symbol MX_Alps_Hybrid:MX-NoLED -> EEMR-TKL-Keyboard-rescue:MX-NoLED-MX_Alps_Hybrid
- MX45: renamed from MX69; footprint (none) -> MX_Only:MXOnly-1U-NoLED; symbol MX_Alps_Hybrid:MX-NoLED -> EEMR-TKL-Keyboard-rescue:MX-NoLED-MX_Alps_Hybrid
- MX46: renamed from MX74; footprint (none) -> MX_Only:MXOnly-1U-NoLED; symbol MX_Alps_Hybrid:MX-NoLED -> EEMR-TKL-Keyboard-rescue:MX-NoLED-MX_Alps_Hybrid
- MX47: renamed from MX79; footprint (none) -> MX_Only:MXOnly-1.5U-NoLED; symbol MX_Alps_Hybrid:MX-NoLED -> EEMR-TKL-Keyboard-rescue:MX-NoLED-MX_Alps_Hybrid
- MX48: renamed from MX82; footprint (none) -> MX_Only:MXOnly-1U-NoLED; symbol MX_Alps_Hybrid:MX-NoLED -> EEMR-TKL-Keyboard-rescue:MX-NoLED-MX_Alps_Hybrid
- MX49: renamed from MX85; footprint (none) -> MX_Only:MXOnly-1U-NoLED; symbol MX_Alps_Hybrid:MX-NoLED -> EEMR-TKL-Keyboard-rescue:MX-NoLED-MX_Alps_Hybrid
- MX5: renamed from MX25; footprint (none) -> MX_Only:MXOnly-1U-NoLED; symbol MX_Alps_Hybrid:MX-NoLED -> EEMR-TKL-Keyboard-rescue:MX-NoLED-MX_Alps_Hybrid
- MX50: renamed from MX87; footprint (none) -> MX_Only:MXOnly-1U-NoLED; symbol MX_Alps_Hybrid:MX-NoLED -> EEMR-TKL-Keyboard-rescue:MX-NoLED-MX_Alps_Hybrid
- MX51: renamed from MX4; footprint (none) -> MX_Only:MXOnly-1.75U-NoLED; symbol MX_Alps_Hybrid:MX-NoLED -> EEMR-TKL-Keyboard-rescue:MX-NoLED-MX_Alps_Hybrid
- MX52: renamed from MX10; footprint (none) -> MX_Only:MXOnly-1U-NoLED; symbol MX_Alps_Hybrid:MX-NoLED -> EEMR-TKL-Keyboard-rescue:MX-NoLED-MX_Alps_Hybrid
- MX53: renamed from MX16; footprint (none) -> MX_Only:MXOnly-1U-NoLED; symbol MX_Alps_Hybrid:MX-NoLED -> EEMR-TKL-Keyboard-rescue:MX-NoLED-MX_Alps_Hybrid
- MX54: renamed from MX22; footprint (none) -> MX_Only:MXOnly-1U-NoLED; symbol MX_Alps_Hybrid:MX-NoLED -> EEMR-TKL-Keyboard-rescue:MX-NoLED-MX_Alps_Hybrid
- MX55: renamed from MX28; footprint (none) -> MX_Only:MXOnly-1U-NoLED; symbol MX_Alps_Hybrid:MX-NoLED -> EEMR-TKL-Keyboard-rescue:MX-NoLED-MX_Alps_Hybrid
- MX56: renamed from MX34; footprint (none) -> MX_Only:MXOnly-1U-NoLED; symbol MX_Alps_Hybrid:MX-NoLED -> EEMR-TKL-Keyboard-rescue:MX-NoLED-MX_Alps_Hybrid
- MX57: renamed from MX40; footprint (none) -> MX_Only:MXOnly-1U-NoLED; symbol MX_Alps_Hybrid:MX-NoLED -> EEMR-TKL-Keyboard-rescue:MX-NoLED-MX_Alps_Hybrid
- MX58: renamed from MX46; footprint (none) -> MX_Only:MXOnly-1U-NoLED; symbol MX_Alps_Hybrid:MX-NoLED -> EEMR-TKL-Keyboard-rescue:MX-NoLED-MX_Alps_Hybrid
- MX59: renamed from MX52; footprint (none) -> MX_Only:MXOnly-1U-NoLED; symbol MX_Alps_Hybrid:MX-NoLED -> EEMR-TKL-Keyboard-rescue:MX-NoLED-MX_Alps_Hybrid
- MX6: renamed from MX31; footprint (none) -> MX_Only:MXOnly-1U-NoLED; symbol MX_Alps_Hybrid:MX-NoLED -> EEMR-TKL-Keyboard-rescue:MX-NoLED-MX_Alps_Hybrid
- MX60: renamed from MX58; footprint (none) -> MX_Only:MXOnly-1U-NoLED; symbol MX_Alps_Hybrid:MX-NoLED -> EEMR-TKL-Keyboard-rescue:MX-NoLED-MX_Alps_Hybrid
- MX61: renamed from MX64; footprint (none) -> MX_Only:MXOnly-1U-NoLED; symbol MX_Alps_Hybrid:MX-NoLED -> EEMR-TKL-Keyboard-rescue:MX-NoLED-MX_Alps_Hybrid
- MX62: renamed from MX70; footprint (none) -> MX_Only:MXOnly-1U-NoLED; symbol MX_Alps_Hybrid:MX-NoLED -> EEMR-TKL-Keyboard-rescue:MX-NoLED-MX_Alps_Hybrid
- MX63: renamed from MX75; footprint (none) -> MX_Only:MXOnly-2.25U-NoLED; symbol MX_Alps_Hybrid:MX-NoLED -> EEMR-TKL-Keyboard-rescue:MX-NoLED-MX_Alps_Hybrid
- MX64: renamed from MX5; footprint (none) -> MX_Only:MXOnly-2.25U-NoLED; symbol MX_Alps_Hybrid:MX-NoLED -> EEMR-TKL-Keyboard-rescue:MX-NoLED-MX_Alps_Hybrid
- MX65: renamed from MX11; footprint (none) -> MX_Only:MXOnly-1U-NoLED; symbol MX_Alps_Hybrid:MX-NoLED -> EEMR-TKL-Keyboard-rescue:MX-NoLED-MX_Alps_Hybrid
- MX66: renamed from MX17; footprint (none) -> MX_Only:MXOnly-1U-NoLED; symbol MX_Alps_Hybrid:MX-NoLED -> EEMR-TKL-Keyboard-rescue:MX-NoLED-MX_Alps_Hybrid
- MX67: renamed from MX23; footprint (none) -> MX_Only:MXOnly-1U-NoLED; symbol MX_Alps_Hybrid:MX-NoLED -> EEMR-TKL-Keyboard-rescue:MX-NoLED-MX_Alps_Hybrid
- MX68: renamed from MX29; footprint (none) -> MX_Only:MXOnly-1U-NoLED; symbol MX_Alps_Hybrid:MX-NoLED -> EEMR-TKL-Keyboard-rescue:MX-NoLED-MX_Alps_Hybrid
- MX69: renamed from MX35; footprint (none) -> MX_Only:MXOnly-1U-NoLED; symbol MX_Alps_Hybrid:MX-NoLED -> EEMR-TKL-Keyboard-rescue:MX-NoLED-MX_Alps_Hybrid
- MX7: renamed from MX37; footprint (none) -> MX_Only:MXOnly-1U-NoLED; symbol MX_Alps_Hybrid:MX-NoLED -> EEMR-TKL-Keyboard-rescue:MX-NoLED-MX_Alps_Hybrid
- MX70: renamed from MX41; footprint (none) -> MX_Only:MXOnly-1U-NoLED; symbol MX_Alps_Hybrid:MX-NoLED -> EEMR-TKL-Keyboard-rescue:MX-NoLED-MX_Alps_Hybrid
- MX71: renamed from MX47; footprint (none) -> MX_Only:MXOnly-1U-NoLED; symbol MX_Alps_Hybrid:MX-NoLED -> EEMR-TKL-Keyboard-rescue:MX-NoLED-MX_Alps_Hybrid
- MX72: renamed from MX53; footprint (none) -> MX_Only:MXOnly-1U-NoLED; symbol MX_Alps_Hybrid:MX-NoLED -> EEMR-TKL-Keyboard-rescue:MX-NoLED-MX_Alps_Hybrid
- MX73: renamed from MX59; footprint (none) -> MX_Only:MXOnly-1U-NoLED; symbol MX_Alps_Hybrid:MX-NoLED -> EEMR-TKL-Keyboard-rescue:MX-NoLED-MX_Alps_Hybrid
- MX74: renamed from MX65; footprint (none) -> MX_Only:MXOnly-1U-NoLED; symbol MX_Alps_Hybrid:MX-NoLED -> EEMR-TKL-Keyboard-rescue:MX-NoLED-MX_Alps_Hybrid
- MX75: renamed from MX71; footprint (none) -> MX_Only:MXOnly-2.75U-NoLED; symbol MX_Alps_Hybrid:MX-NoLED -> EEMR-TKL-Keyboard-rescue:MX-NoLED-MX_Alps_Hybrid
- MX77: renamed from MX6; footprint (none) -> MX_Only:MXOnly-1.25U-NoLED; symbol MX_Alps_Hybrid:MX-NoLED -> EEMR-TKL-Keyboard-rescue:MX-NoLED-MX_Alps_Hybrid
- MX78: renamed from MX12; footprint (none) -> MX_Only:MXOnly-1.25U-NoLED; symbol MX_Alps_Hybrid:MX-NoLED -> EEMR-TKL-Keyboard-rescue:MX-NoLED-MX_Alps_Hybrid
- MX79: renamed from MX18; footprint (none) -> MX_Only:MXOnly-1.25U-NoLED; symbol MX_Alps_Hybrid:MX-NoLED -> EEMR-TKL-Keyboard-rescue:MX-NoLED-MX_Alps_Hybrid
- MX8: renamed from MX43; footprint (none) -> MX_Only:MXOnly-1U-NoLED; symbol MX_Alps_Hybrid:MX-NoLED -> EEMR-TKL-Keyboard-rescue:MX-NoLED-MX_Alps_Hybrid
- MX80: renamed from MX24; footprint (none) -> MX_Only:MXOnly-6.25U-NoLED; symbol MX_Alps_Hybrid:MX-NoLED -> EEMR-TKL-Keyboard-rescue:MX-NoLED-MX_Alps_Hybrid
- MX81: renamed from MX30; footprint (none) -> MX_Only:MXOnly-1.25U-NoLED; symbol MX_Alps_Hybrid:MX-NoLED -> EEMR-TKL-Keyboard-rescue:MX-NoLED-MX_Alps_Hybrid
- MX82: renamed from MX36; footprint (none) -> MX_Only:MXOnly-1.25U-NoLED; symbol MX_Alps_Hybrid:MX-NoLED -> EEMR-TKL-Keyboard-rescue:MX-NoLED-MX_Alps_Hybrid
- MX83: renamed from MX42; footprint (none) -> MX_Only:MXOnly-1.25U-NoLED; symbol MX_Alps_Hybrid:MX-NoLED -> EEMR-TKL-Keyboard-rescue:MX-NoLED-MX_Alps_Hybrid
- MX84: renamed from MX48; footprint (none) -> MX_Only:MXOnly-1.25U-NoLED; symbol MX_Alps_Hybrid:MX-NoLED -> EEMR-TKL-Keyboard-rescue:MX-NoLED-MX_Alps_Hybrid
- MX85: renamed from MX54; footprint (none) -> MX_Only:MXOnly-1U-NoLED; symbol MX_Alps_Hybrid:MX-NoLED -> EEMR-TKL-Keyboard-rescue:MX-NoLED-MX_Alps_Hybrid
- MX86: renamed from MX60; footprint (none) -> MX_Only:MXOnly-1U-NoLED; symbol MX_Alps_Hybrid:MX-NoLED -> EEMR-TKL-Keyboard-rescue:MX-NoLED-MX_Alps_Hybrid
- MX87: renamed from MX66; footprint (none) -> MX_Only:MXOnly-1U-NoLED; symbol MX_Alps_Hybrid:MX-NoLED -> EEMR-TKL-Keyboard-rescue:MX-NoLED-MX_Alps_Hybrid
- MX9: renamed from MX49; footprint (none) -> MX_Only:MXOnly-1U-NoLED; symbol MX_Alps_Hybrid:MX-NoLED -> EEMR-TKL-Keyboard-rescue:MX-NoLED-MX_Alps_Hybrid
- R1: renamed from R3; footprint (none) -> Resistor_SMD:R_0805_2012Metric_Pad1.15x1.40mm_HandSolder
- R2, R6: footprint (none) -> Resistor_SMD:R_0805_2012Metric_Pad1.15x1.40mm_HandSolder
- R3: renamed from R1; footprint (none) -> Resistor_SMD:R_0805_2012Metric_Pad1.15x1.40mm_HandSolder
- R4: renamed from R5; footprint (none) -> Resistor_SMD:R_0805_2012Metric_Pad1.15x1.40mm_HandSolder
- R5: renamed from R4; footprint (none) -> Resistor_SMD:R_0805_2012Metric_Pad1.15x1.40mm_HandSolder
- SW1: footprint (none) -> random-keyboard-parts:SKQG-1155865
- USB1: footprint (none) -> Type-C:HRO-TYPE-C-31-M-12-HandSoldering; symbol Type-C:HRO-TYPE-C-31-M-12 -> EEMR-TKL-Keyboard-rescue:HRO-TYPE-C-31-M-12-Type-C
- Y1: footprint (none) -> Crystal:Crystal_SMD_3225-4Pin_3.2x2.5mm_HandSoldering
- renumbered D55 to D10, D61 to D11, D67 to D12, D72 to D13, D77 to D14, D80 to D15, D83 to D16, D2 to D17, D8 to D18, D14 to D19, D7 to D2, D26 to D21, D32 to D22, D38 to D23, D44 to D24, D50 to D25, D56 to D26, D62 to D27, D68 to D28, D73 to D29, D13 to D3, D78 to D30, D81 to D31, D84 to D32, D86 to D33, D3 to D34, D9 to D35, D15 to D36, D21 to D37, D27 to D38, D33 to D39, D19 to D4, D39 to D40, D45 to D41, D51 to D42, D57 to D43, D63 to D44, D69 to D45, D74 to D46, D79 to D47, D82 to D48, D85 to D49, D25 to D5, D87 to D50, D4 to D51, D10 to D52, D16 to D53, D22 to D54, D28 to D55, D34 to D56, D40 to D57, D46 to D58, D52 to D59, D31 to D6, D58 to D60, D64 to D61, D70 to D62, D75 to D63, D5 to D64, D11 to D65, D17 to D66, D23 to D67, D29 to D68, D35 to D69, D37 to D7, D41 to D70, D47 to D71, D53 to D72, D59 to D73, D65 to D74, D71 to D75, D6 to D77, D12 to D78, D18 to D79, D43 to D8, D24 to D80, D30 to D81, D36 to D82, D42 to D83, D48 to D84, D54 to D85, D60 to D86, D66 to D87, D49 to D9
Other:
- moved on the sheet: D10, D11, D12, D13, D14, D15, D16, D2, D3, D4, D5, D6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
